File: production/kicad/lira.kicad_pcb (KiCad board)
At the start: 2 copper layers, 334.6 x 100.2 mm, 226 parts, among them J1 USB-C, J2 battery JST-PH, J3 PJ-320D-4A, Q1 SI2301CDS, SW1 7, SW10 T, SW101 JS102011SAQN, SW102 reset, SW11 Y, SW12 U, SW13 I, SW14 O, SW15 P, SW16 \, SW17 delete, SW18 4, SW19 5, SW2 8, SW20 6, SW21 +, SW22 tab, SW23 A, SW24 S, SW25 D, SW26 F, SW27 G, SW28 H, SW29 J, SW3 9, SW30 K, SW31 L, SW32 ;, SW33 return, SW34 1, SW35 2, SW36 3, SW37 enter, SW38 shift, SW39 Z, SW4 −, SW40 X, SW41 C, SW42 V, SW43 B, SW44 N, SW45 M, SW46 ,, SW47 ., SW48 shift, SW49 fn, SW5 esc, SW50 0, SW51 ., SW52 option, SW53 ⌘, SW54 space, SW55 space, SW56 ⌘, SW57 option, SW6 Q, SW7 W, SW8 E, SW9 R, U1 E73-2G4M08S1C, U2 MCP73831, U3 AP2112K-3.3, U4 USBLC6-2SC6, U5 CH334P, U6 CM108B, U7 TPA6132A2, U8 TPS22919, Y1 32.768kHz, Y2 12MHz

Commit message: Right-size the ground stitching: 916 -> 318 vias (5mm strip / 12mm key field), drop single-layer vias; no electrical change (DRC 0, ERC 0, netlist match, 51 checks pass)
Routing:
- net GND: vias 758 -> 161
- net VBUS: vias 13 -> 12
