File: production/kicad/lira.kicad_pcb (KiCad board)
At the start: 2 copper layers, 334.6 x 100.2 mm, 226 parts, among them J1 USB-C, J2 battery JST-PH, J3 PJ-320D-4A, Q1 SI2301CDS, SW1 7, SW10 T, SW101 JS102011SAQN, SW102 reset, SW11 Y, SW12 U, SW13 I, SW14 O, SW15 P, SW16 \, SW17 delete, SW18 4, SW19 5, SW2 8, SW20 6, SW21 +, SW22 tab, SW23 A, SW24 S, SW25 D, SW26 F, SW27 G, SW28 H, SW29 J, SW3 9, SW30 K, SW31 L, SW32 ;, SW33 return, SW34 1, SW35 2, SW36 3, SW37 enter, SW38 shift, SW39 Z, SW4 −, SW40 X, SW41 C, SW42 V, SW43 B, SW44 N, SW45 M, SW46 ,, SW47 ., SW48 shift, SW49 fn, SW5 esc, SW50 0, SW51 ., SW52 option, SW53 ⌘, SW54 space, SW55 space, SW56 ⌘, SW57 option, SW6 Q, SW7 W, SW8 E, SW9 R, U1 E73-2G4M08S1C, U2 MCP73831, U3 AP2112K-3.3, U4 USBLC6-2SC6, U5 CH334P, U6 CM108B, U7 TPA6132A2, U8 TPS22919, Y1 32.768kHz, Y2 12MHz

Commit message: Rework and re-route the board
Circuit and board:
- MAJ-1: reverse-battery P-MOSFET Q2 (SI2301) between the battery connector
  and the switch, gate to GND: a reversed cell finds it off
- the hub (V5 abs max 5.5 V) on its own 3.3 V regulator U9 from VBUS
  (CH334 datasheet 6.4); SMF5.0A TVS at the receptacle; C107 through 1 ohm
  (R126) damps the hot-plug ring without adding capacitance
- MIN-8: TPS7A0233 (25 nA) instead of the AP2112K (55 uA); C103 4.7 uF
  to stay inside its 1-22 uF output range
- MIN-1/2: C137 470 -> 100 nF, R124 33k in series with the amplifier's EN
- MIN-5: the codec's PDSW switches the amplifier off in USB suspend (Q3)
- MIN-9/10: ground vias ringed around the module and the charger, and a via
  at the charger's ground pin (finish step)
- DFM: no via in the amplifier's exposed pad; the hub's paste is a frame
  clear of its ground via
- placement data rotations for the new part types

Firmware: P1.02 standard drive; REG1 DC/DC on (inductors inside the
module); low-battery cut-off (System OFF below 3.40 V without USB).

Checks: new P07 (reverse battery), U04 (VBUS), A15 (suspend); L01-L03, H01,
C02, A14 extended; mutation-tested. Schematic on A1 with room for the
notes; ERC 0 warnings. .

Docs updated.
Parts:
- added D108: SMF5.0A, D_SOD-123F, B.Cu at (103.2, 14.0)
- added Q2: SI2301CDS, SOT-23, B.Cu at (72.5, 14.5)
- added Q3: 2N7002, SOT-23, B.Cu at (225.2, 12.1)
- added R124: 33k, R_0603_1608Metric, B.Cu at (218.3, 24.0)
- added R125: 100k, R_0603_1608Metric, B.Cu at (228.6, 12.3)
- added R126: 1, R_0603_1608Metric, B.Cu at (100.5, 21.5)
- added U9: TPS7A0233, SOT-23-5, B.Cu at (120.0, 19.6)
- C103: value 10uF -> 4.7uF
- C137: value 470nF -> 100nF
- U3: value AP2112K-3.3 -> TPS7A0233
- moved C110 8.32 mm to (119.8, 16.0), turned to 0 degrees
- moved C137 0.90 mm to (218.8, 27.3)
Connections:
- C107 pad 1: VBUS -> VBUS_DAMP
- J2 pad 1: BAT+ -> BAT_IN
- U5 pad 15: VBUS -> HUB_3V3
- U6 pad 40: (no net) -> CM_PDSW
- U7 pad 13: AMP_EN -> AMP_ENI
Routing:
- net GND: track 401.2 -> 480.3 mm, vias 161 -> 183
- net CM_PDSW: track 0.00 -> 53.6 mm, vias 0 -> 2
- net COL5: track 126.7 -> 91.5 mm
- net ROW3: track 398.1 -> 375.9 mm
- net AMP_EN: track 12.2 -> 31.0 mm, vias 0 -> 4
- net VIN: track 47.2 -> 34.4 mm, vias 0 -> 2
- net COL14: track 233.9 -> 221.2 mm, vias 2 -> 0
- net LOR: track 9.88 -> 21.9 mm, vias 2 -> 6
- net ROW1: track 407.0 -> 396.8 mm
- net HPL2: track 36.6 -> 46.1 mm
- net SD24: track 18.9 -> 10.1 mm
- net BAT_IN: track 0.00 -> 8.00 mm
- net VBUS: track 223.6 -> 231.1 mm, vias 12 -> 11
- net COL3: track 133.5 -> 141.0 mm
- net SD52: track 18.9 -> 11.8 mm
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- added copper zone on F.Cu, net AMP_EN
- added copper zone on B.Cu, net AMP_G0
- added copper zone on B.Cu, net BAT_IN
- added copper zone on B.Cu, net CM_PDSW
- added copper zone on F.Cu, net CM_PDSW
- added copper zone on F.Cu, net MIC
- added copper zone on B.Cu, net SD10
- added copper zone on B.Cu, net SD3
- added copper zone on B.Cu, net SD38
- added copper zone on B.Cu, net SD5
- added copper zone on B.Cu, net SD50
- added copper zone on F.Cu, net STAT
- added copper zone on B.Cu, net VBUS_DAMP
- removed copper zone on B.Cu, net AUD_AVDD
- removed copper zone on F.Cu, net BAT+
- removed copper zone on F.Cu, net BAT_SENSE
- removed copper zone on B.Cu, net CC1
- removed copper zone on B.Cu, net CM_MODE
- removed copper zone on F.Cu, net CM_MODE
- removed copper zone on F.Cu, net COL14
- removed copper zone on F.Cu, net COL15
- removed copper zone on F.Cu, net COL4
- removed copper zone on B.Cu, net HPL2
- removed copper zone on B.Cu, net HUB_3V3
- removed copper zone on B.Cu, net SD44
- removed copper zone on B.Cu, net XL2
Other:
- board text added: "LIRA rev B"
- board text removed: "LIRA rev A"
