File: production/kicad/lira.kicad_pcb (KiCad board)
At the start: 2 copper layers, 334.6 x 100.2 mm, 226 parts, among them J1 USB-C, J2 battery JST-PH, J3 PJ-320D-4A, Q1 SI2301CDS, SW1 7, SW10 T, SW101 JS102011SAQN, SW102 reset, SW11 Y, SW12 U, SW13 I, SW14 O, SW15 P, SW16 \, SW17 delete, SW18 4, SW19 5, SW2 8, SW20 6, SW21 +, SW22 tab, SW23 A, SW24 S, SW25 D, SW26 F, SW27 G, SW28 H, SW29 J, SW3 9, SW30 K, SW31 L, SW32 ;, SW33 return, SW34 1, SW35 2, SW36 3, SW37 enter, SW38 shift, SW39 Z, SW4 −, SW40 X, SW41 C, SW42 V, SW43 B, SW44 N, SW45 M, SW46 ,, SW47 ., SW48 shift, SW49 fn, SW5 esc, SW50 0, SW51 ., SW52 option, SW53 ⌘, SW54 space, SW55 space, SW56 ⌘, SW57 option, SW6 Q, SW7 W, SW8 E, SW9 R, U1 E73-2G4M08S1C, U2 MCP73831, U3 AP2112K-3.3, U4 USBLC6-2SC6, U5 CH334P, U6 CM108B, U7 TPA6132A2, U8 TPS22919, Y1 32.768kHz, Y2 12MHz

Commit message: rp2040: complete the wired variant (RP2040, USB only, no battery)
Same keyboard, case, plate, sound card and keymap as main; the nRF52840 module, battery, charger,
power path and power switch are replaced by a Raspberry Pi RP2040 with its minimum circuit.

- circuit: RP2040 per "Hardware design with RP2040" (ABM8-272-T3 12 MHz, 2 x 15 pF, 1k on XOUT;
  W25Q128JV, SOIC-8 208 mil; 100 nF per supply pin, 1 uF on VREG_VIN/VOUT; BOOT and RESET
  buttons; 27 ohm USB series); fixes from the WIP: VREG_VIN was unconnected, flash footprint was
  150 mil. Sound card identical to main except the TPS22919 ON / amp EN network driven by VBUS
  (keeps the soft start), refs aligned with main
- PCB: new RP2040 block placement; Fine net class (0.2 mm) for the 0.4 mm-pitch pads, matrix lines
  widened back to 0.3 mm after routing; pre-drawn core supply (under the chip), SWD lines, hub
  crystal, amp VDD and load-switch ground; DRC 0 violations, 0 unconnected
- finish_pcb: removed vias kept alive (SWIG use-after-free), geometric via pruning; gen_pcb: no
  stale .kicad_pro loaded, so a rebuild equals a clean build
- schematic regenerated (ERC 0 errors), netlist match; independent checker extended for the
  RP2040 (Q01-Q12): 42 PASS, 0 FAIL, 3 WARN; main's netlist unchanged
- case: no battery pocket, paperclip hole to BOOT; fit check 0 FAIL, 3 WARN (as main)
- firmware: RMK 0.9 + Vial on the RP2040 (embassy-rp, boot2 W25Q080), no BLE / audio gate
- docs: README, build guide, source README, production regenerated; usb/ scaffold folded in
Parts:
- removed C101: 10uF, C_0603_1608Metric
- removed C104: 10nF, C_0603_1608Metric
- removed C105, C106: 18pF, C_0603_1608Metric
- removed C107: 4.7uF, C_0603_1608Metric
- removed C109: 100nF, C_0603_1608Metric
- removed D101: B5819W, D_SOD-123
- removed D102: LED white, LED_0603_1608Metric
- removed J2: battery JST-PH, JST_PH_S2B-PH-SM4-TB_1x02-1MP_P2.00mm_Horizontal
- removed JP1: charge 200 mA, SolderJumper-2_P1.3mm_Open_RoundedPad1.0x1.5mm
- removed JP2: switch bypass, SolderJumper-2_P1.3mm_Open_RoundedPad1.0x1.5mm
- removed Q1: SI2301CDS, SOT-23
- removed R101, R117: 100k, R_0603_1608Metric
- removed R102: 1k, R_0603_1608Metric
- removed R103, R104: 10k, R_0603_1608Metric
- removed R105, R106: 10M, R_0603_1608Metric
- removed TP7: VBAT, TestPoint_Pad_D1.5mm
- removed TP8: VIN, TestPoint_Pad_D1.5mm
- added C1: 100nF, C_0603_1608Metric, B.Cu at (141.0, 19.5)
- added C10: 100nF, C_0603_1608Metric, B.Cu at (134.6, 15.1)
- added C11: 1uF, C_0603_1608Metric, B.Cu at (125.0, 15.1)
- added C12: 1uF, C_0603_1608Metric, B.Cu at (126.6, 15.1)
- added C13: 15pF, C_0603_1608Metric, B.Cu at (144.2, 28.6)
- added C14: 15pF, C_0603_1608Metric, B.Cu at (138.5, 32.7)
- added C15: 100nF, C_0603_1608Metric, B.Cu at (149.4, 17.6)
- added C2: 100nF, C_0603_1608Metric, B.Cu at (144.5, 23.5)
- added C3: 100nF, C_0603_1608Metric, B.Cu at (136.4, 29.3)
- added C4: 100nF, C_0603_1608Metric, B.Cu at (125.5, 23.5)
- added C5: 100nF, C_0603_1608Metric, B.Cu at (129.0, 19.3)
- added C6: 100nF, C_0603_1608Metric, B.Cu at (133.0, 15.1)
- added C7: 100nF, C_0603_1608Metric, B.Cu at (131.4, 15.1)
- added C8: 100nF, C_0603_1608Metric, B.Cu at (123.4, 15.1)
- added C9: 100nF, C_0603_1608Metric, B.Cu at (134.9, 29.3)
- added R1: 1k, R_0603_1608Metric, B.Cu at (137.9, 29.3)
- added R2: 10k, R_0603_1608Metric, B.Cu at (144.2, 18.2)
- added R3: 1k, R_0603_1608Metric, B.Cu at (152.0, 15.5)
- added R4: 10k, R_0603_1608Metric, B.Cu at (160.2, 15.5)
- added R5: 27, R_0603_1608Metric, B.Cu at (129.8, 15.1)
- added R6: 27, R_0603_1608Metric, B.Cu at (128.2, 15.1)
- SW101: value JS102011SAQN -> BOOT; footprint SW_SPDT_CK_JS102011SAQN -> SW-SMD_4P-L5.1-W5.1-P3.70-LS6.5-TL_H1.5
- SW102: value reset -> RESET
- U1: value E73-2G4M08S1C -> RP2040; footprint WIRELM-SMD_E73-2G4M08S1C -> QFN-56-1EP_7x7mm_P0.4mm_EP3.2x3.2mm
- U2: value MCP73831 -> W25Q128JVS; footprint SOT-23-5 -> SOIC-8_5.3x5.3mm_P1.27mm
- Y1: value 32.768kHz -> 12MHz; footprint Crystal_SMD_3215-2Pin_3.2x1.5mm -> Crystal_SMD_3225-4Pin_3.2x2.5mm
- moved SW101 68.1 mm to (156.0, 15.5)
- moved U2 49.4 mm to (143.8, 14.3)
- moved TP2 19.0 mm to (134.0, 32.3)
- moved TP1 15.8 mm to (132.0, 32.3)
- moved C103 13.8 mm to (123.2, 18.9), turned to 0 degrees
- moved TP4 11.6 mm to (128.0, 32.3)
- moved SW102 10.7 mm to (164.5, 15.5)
- moved TP3 9.42 mm to (120.8, 15.1)
- moved TP5 8.61 mm to (130.0, 32.3)
- moved Y1 3.67 mm to (140.9, 29.7), turned to -90 degrees
- moved U1 1.50 mm to (135.0, 22.5), turned to 180 degrees
Connections:
- C102 pad 1: VIN -> VBUS
- D104 pad 1: AUD_EN -> VBUS
- R113 pad 1: AUD_EN -> VBUS
- SW101 pad 1: BAT+ -> BOOT
- SW101 pad 2: VBAT -> (no net)
- U1 pad 1: (no net) -> 3V3
- U1 pad 10: ROW2 -> 3V3
- U1 pad 11: XL1 -> COL8
- U1 pad 12: COL11 -> COL7
- U1 pad 13: XL2 -> ROW0
- U1 pad 14: COL16 -> COL6
- U1 pad 15: ROW3 -> (no net)
- U1 pad 16: COL10 -> (no net)
- U1 pad 17: ROW1 -> (no net)
- U1 pad 18: COL9 -> (no net)
- U1 pad 19: 3V3 -> GND
- U1 pad 2: (no net) -> COL15
- U1 pad 20: COL8 -> XIN
- U1 pad 21: GND -> XOUT
- U1 pad 22: COL7 -> 3V3
- U1 pad 23: 3V3 -> 1V1
- U1 pad 24: GND -> SWCLK
- U1 pad 25: (no net) -> SWDIO
- U1 pad 27: VBUS -> (no net)
- U1 pad 28: COL6 -> (no net)
- U1 pad 29: MCU_DN -> ROW2
- U1 pad 3: COL15 -> COL14
- U1 pad 30: COL5 -> ROW3
- U1 pad 31: MCU_DP -> ROW1
- U1 pad 32: COL4 -> COL5
- U1 pad 33: COL3 -> 3V3
- U1 pad 34: COL2 -> COL4
- U1 pad 35: COL1 -> COL3
- U1 pad 36: COL0 -> COL2
- U1 pad 37: SWDIO -> COL1
- U1 pad 38: AUD_EN -> COL0
- U1 pad 39: SWCLK -> LED_RED
- U1 pad 4: COL14 -> COL13
- U1 pad 40: LED_RED -> (no net)
- U1 pad 42: (no net) -> 3V3
- U1 pad 43: (no net) -> 3V3
- U1 pad 5: GND -> COL12
- U1 pad 6: COL13 -> COL11
- U1 pad 7: COL12 -> COL16
- U1 pad 8: ROW0 -> COL10
- U1 pad 9: BAT_SENSE -> COL9
- U2 pad 1: STAT -> QSPI_SS
- U2 pad 2: GND -> QSPI_SD1
- U2 pad 3: VBAT -> QSPI_SD2
- U2 pad 4: VBUS -> GND
- U2 pad 5: PROG -> QSPI_SD0
- U3 pad 1: VIN -> VBUS
- U3 pad 3: VIN -> VBUS
- U8 pad 3: AUD_EN -> VBUS
- Y1 pad 1: XL1 -> XIN
- Y1 pad 2: XL2 -> GND
Routing:
- net VBAT: track 111.1 -> 0.00 mm, vias 4 -> 0
- net 3V3: track 53.0 -> 158.8 mm, vias 3 -> 6
- net AUD_EN: track 103.3 -> 0.00 mm, vias 4 -> 0
- net ROW0: track 389.7 -> 482.7 mm, vias 20 -> 14
- net GND: track 401.2 -> 486.9 mm, vias 161 -> 187
- net VIN: track 47.2 -> 0.00 mm
- net RP_DP: track 0.00 -> 39.8 mm, vias 0 -> 6
- net 1V1: track 0.00 -> 34.1 mm, vias 0 -> 2
- net VBUS: track 223.6 -> 191.3 mm, vias 12 -> 9
- net BAT+: track 26.7 -> 0.00 mm, vias 2 -> 0
- net COL5: track 126.7 -> 100.4 mm, vias 2 -> 0
- net RESET: track 33.5 -> 54.6 mm, vias 2 -> 0
- net AUD_AVDD: track 20.9 -> 40.0 mm, vias 2 -> 4
- net COL6: track 89.5 -> 108.3 mm
- net QSPI_SS: track 0.00 -> 18.3 mm, vias 0 -> 3
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- added copper zone on B.Cu, net 1V1
- added copper zone on F.Cu, net 1V1
- added copper zone on B.Cu, net BOOT
- added copper zone on B.Cu, net CM_MSEL
- added copper zone on F.Cu, net COL12
- added copper zone on F.Cu, net COL13
- added copper zone on B.Cu, net HUB_XO
- added copper zone on F.Cu, net MIC
- added copper zone on F.Cu, net QSPI_SCLK
- added copper zone on B.Cu, net QSPI_SD0
- added copper zone on F.Cu, net QSPI_SD0
- added copper zone on B.Cu, net QSPI_SD1
- added copper zone on B.Cu, net QSPI_SD2
- added copper zone on F.Cu, net QSPI_SD3
- added copper zone on B.Cu, net QSPI_SS
- added copper zone on F.Cu, net QSPI_SS
- added copper zone on B.Cu, net RP_DP
- added copper zone on F.Cu, net RP_DP
- added copper zone on B.Cu, net SD10
- added copper zone on B.Cu, net SD13
- added copper zone on B.Cu, net SD2
- added copper zone on B.Cu, net SD3
- added copper zone on B.Cu, net SD33
- added copper zone on B.Cu, net SD38
- added copper zone on B.Cu, net SD5
- added copper zone on B.Cu, net SD50
- added copper zone on B.Cu, net SWDIO
- added copper zone on B.Cu, net XIN
- added copper zone on F.Cu, net XIN
- added copper zone on B.Cu, net XOUT
- removed copper zone on B.Cu, net AMP_INL
- removed copper zone on B.Cu, net AMP_INR
- removed copper zone on B.Cu, net AUD_EN
- removed copper zone on F.Cu, net AUD_EN
- removed copper zone on B.Cu, net BAT+
- removed copper zone on F.Cu, net BAT+
- removed copper zone on B.Cu, net BAT_SENSE
- removed copper zone on F.Cu, net BAT_SENSE
- removed copper zone on B.Cu, net CC1
- removed copper zone on B.Cu, net CM_MODE
- removed copper zone on F.Cu, net CM_MODE
- removed copper zone on F.Cu, net COL0
- removed copper zone on F.Cu, net COL1
- removed copper zone on F.Cu, net COL2
- removed copper zone on F.Cu, net COL3
- removed copper zone on F.Cu, net COL5
- removed copper zone on F.Cu, net LOL
- removed copper zone on B.Cu, net LOR
- removed copper zone on B.Cu, net PROG
- removed copper zone on B.Cu, net PROG_ALT
- removed copper zone on F.Cu, net RESET
- removed copper zone on B.Cu, net STAT
- removed copper zone on B.Cu, net VBAT
- removed copper zone on F.Cu, net VBAT
- removed copper zone on B.Cu, net VIN
- removed copper zone on B.Cu, net VREF
- removed copper zone on B.Cu, net XL2
Other:
- board text added: "BOOT"
- board text added: "LIRA wired rev A"
- board text removed: "+"
- board text removed: "-"
- board text removed: "200mA"
- board text removed: "CHG"
- board text removed: "LIRA rev A"
- board text removed: "SW BYP"
- board text removed: "VBAT"
- board text removed: "VIN"
