File: production/kicad/schematic/lira.kicad_sch (KiCad schematic)
At the start: 211 parts, among them J1 USB-C, J2 battery JST-PH, J3 PJ-320D-4A, Q1 SI2301CDS, SW1 7, SW10 T, SW101 JS102011SAQN, SW102 reset, SW11 Y, SW12 U, SW13 I, SW14 O, SW15 P, SW16 \, SW17 delete, SW18 4, SW19 5, SW2 8, SW20 6, SW21 +, SW22 tab, SW23 A, SW24 S, SW25 D, SW26 F, SW27 G, SW28 H, SW29 J, SW3 9, SW30 K, SW31 L, SW32 ;, SW33 return, SW34 1, SW35 2, SW36 3, SW37 enter, SW38 shift, SW39 Z, SW4 −, SW40 X, SW41 C, SW42 V, SW43 B, SW44 N, SW45 M, SW46 ,, SW47 ., SW48 shift, SW49 fn, SW5 esc, SW50 0, SW51 ., SW52 option, SW53 ⌘, SW54 space, SW55 space, SW56 ⌘, SW57 option, SW6 Q, SW7 W, SW8 E, SW9 R, U1 E73-2G4M08S1C, U2 MCP73831, U3 AP2112K-3.3, U4 USBLC6-2SC6, U5 CH334P, U6 CM108B, U7 TPA6132A2, U8 TPS22919, Y1 32.768kHz, Y2 12MHz

Commit message: Fix placement data, silkscreen, firmware and docs
Supply and placement (blocking before an order):
- Hot-swap socket C2803348 is discontinued (0 stock): replaced by C41430893
  in the BOM, schematic, netlist and checks
- cpl.csv: rotations converted to JLCPCB's convention (per-part LCSC
  footprint angle, bottom side 180 - angle) and origin offsets for J1, J3
  and SW101

Board (silkscreen only; tracks, vias and placement unchanged, DRC 0 errors):
- every label >= 1.0 mm; SW BYP, -6dB, VBAT, CHG and CAPS moved off pads
  and apart, in the generator and in the published board

Firmware:
- random Vial keyboard UID; fn+T (forget the paired host) removed from
  the default keymap; memory.x stops the link before RMK's storage;
  Cargo.toml metadata

Build: placement step and one datasheet check made deterministic.

Docs: README, guide and production README corrected (screws, ears, print
orientation, JLCPCB options, bench checks, licences) and
Parts:
- SW1, SW10, SW11, SW12, SW13, SW14, SW15, SW16, SW17, SW18, SW19, SW2, SW20, SW21, SW22, SW23, SW24, SW25, SW26, SW27, SW28, SW29, SW3, SW30, SW31, SW32, SW33, SW34, SW35, SW36, SW37, SW38, SW39, SW4, SW40, SW41, SW42, SW43, SW44, SW45, SW46, SW47, SW48, SW49, SW5, SW50, SW51, SW52, SW53, SW54, SW55, SW56, SW57, SW6, SW7, SW8, SW9: LCSC C2803348 -> C41430893

Commit message: Rework and re-route the board
Circuit and board:
- MAJ-1: reverse-battery P-MOSFET Q2 (SI2301) between the battery connector
  and the switch, gate to GND: a reversed cell finds it off
- the hub (V5 abs max 5.5 V) on its own 3.3 V regulator U9 from VBUS
  (CH334 datasheet 6.4); SMF5.0A TVS at the receptacle; C107 through 1 ohm
  (R126) damps the hot-plug ring without adding capacitance
- MIN-8: TPS7A0233 (25 nA) instead of the AP2112K (55 uA); C103 4.7 uF
  to stay inside its 1-22 uF output range
- MIN-1/2: C137 470 -> 100 nF, R124 33k in series with the amplifier's EN
- MIN-5: the codec's PDSW switches the amplifier off in USB suspend (Q3)
- MIN-9/10: ground vias ringed around the module and the charger, and a via
  at the charger's ground pin (finish step)
- DFM: no via in the amplifier's exposed pad; the hub's paste is a frame
  clear of its ground via
- placement data rotations for the new part types

Firmware: P1.02 standard drive; REG1 DC/DC on (inductors inside the
module); low-battery cut-off (System OFF below 3.40 V without USB).

Checks: new P07 (reverse battery), U04 (VBUS), A15 (suspend); L01-L03, H01,
C02, A14 extended; mutation-tested. Schematic on A1 with room for the
notes; ERC 0 warnings. .

Docs updated.
Parts:
- removed U3: AP2112K-3.3, Package_TO_SOT_SMD:SOT-23-5, symbol Regulator_Linear:AP2112K-3.3
- added D108: SMF5.0A, Diode_SMD:D_SOD-123F, symbol Device:D_Zener
- added Q2: SI2301CDS, Package_TO_SOT_SMD:SOT-23, symbol Transistor_FET:AO3401A
- added Q3: 2N7002, Package_TO_SOT_SMD:SOT-23, symbol Transistor_FET:2N7002
- added R124: 33k, Resistor_SMD:R_0603_1608Metric, symbol Device:R
- added R125: 100k, Resistor_SMD:R_0603_1608Metric, symbol Device:R
- added R126: 1, Resistor_SMD:R_0603_1608Metric, symbol Device:R
- added U3, U9: TPS7A0233, Package_TO_SOT_SMD:SOT-23-5, symbol lira:TPS7A02
- C103: value 10uF -> 4.7uF; LCSC C19702 -> C19666
- C137: value 470nF -> 100nF; LCSC C1623 -> C14663
Connections:
- net 3V3: now also U3.5 (OUT)
- net AMP_EN: now also Q3.3 (D), R124.1; no longer U7.13 (EN)
- net AUD_5V: now also R125.2
- net BAT+: now also Q2.2 (S); no longer J2.1 (Pin_1)
- net GND: now also D108.2 (A), Q2.1 (G), Q3.2 (S), U3.2 (GND), U9.2 (GND)
- net HUB_3V3: now also U5.15 (V5), U9.5 (OUT)
- net VBUS: now also D108.1 (K), R126.1, U9.1 (IN), U9.3 (EN); no longer C107.1, U5.15 (V5)
- net VIN: now also U3.1 (IN), U3.3 (EN)
- net CM_PDSW: now reaches U6.40 (PDSW)
- net CM_PDSW: now also Q3.1 (G), R125.1
- new net AMP_ENI: R124.2, U7.13 (EN)
- new net BAT_IN: J2.1 (Pin_1), Q2.3 (D)
- new net VBUS_DAMP: C107.1, R126.2
Other:
- note added: "1. Second regulator (switched 3.3 V for external devices, P0.12 enable) omitted: nothing external to power."
- note added: "11. C108 1 uF at the regulator output and C109 100 nF at the module: the 4.7 uF C103 sits at the module's supply pins (VDD / VDDH), 25 mm away (the module has about 12 uF inside: the TPS7A02 allows 1-22 uF on its output). C102 on VIN is 1 uF instead of 10 uF: together they keep the capacitance charged at USB attach near USB 2.0's 10 uF."
- note added: "15. Reverse-battery P-MOSFET Q2 (SI2301) between the battery connector and the switch, gate to GND: a cell plugged in the wrong way round finds it off (its body diode blocks), so the charger's VBAT pin never sees a negative voltage; the right way round it is on (Vgs = -Vbat) and charging goes through it."
- note added: "16. Regulator TPS7A0233 (25 nA quiescent, 200 mA) instead of the AP2112K (55 uA): same SOT-23-5 pins (IN, GND, EN, NC, OUT); the 3.3 V rail needs < 50 mA (module, status LED)."
- note added: "17. VBUS: an SMF5.0A TVS at the receptacle, and C107 (4.7 uF) through 1 ohm: a ceramic-only VBUS rings on hot plug to 6-8 V through the cable's inductance (simulated, 0.5-1 uH); damped, 5.0-6.6 V, without adding capacitance."
- note added: "3. Amplifier off in USB suspend: the codec's PDSW (open drain, low in operation, open in suspend; app note 1.50) with a 100k pull-up to AUD_5V drives"
- note added: "4. Hub supply: V5 and VDD33 both on a 3.3 V regulator (TPS7A0233) fed from VBUS (CH334 datasheet 6.4), instead of V5 on VBUS: V5's absolute maximum is"
- note added: "5. Microphone: bias 1.2k + 2.2k (demo board 2.2k + 8.2k, for PC microphones) for phone headsets (Android: 1.8-2.9 V through 2.2k); 1k in series before"
- note added: "5.5 V and a USB hot plug rings above it; the regulator's input is rated 6.5 V. The regulator is on only with VBUS (the hub draws nothing from the"
- note added: "6. The demo board's two 10 nF capacitors DVDD - DREG18 and DVDD - DREG33 ('close to IC', for ESD) are fitted."
- note added: "7. The amplifier's SGND (pin 15) is grounded at the amplifier (its ground pad and a via into the top ground plane), not on a track of its own to the"
- note added: "8. The four mode jumpers are also strapped with 10k (MODE/ADSEL low, PWRSEL/MSEL high to DREG33) on top of the chip's internal pulls. D105-D107 are"
- note added: "C107: VBUS bypass (deviation 10), damped by R126 (deviation 17)"
- note added: "V5 = VDD33 = 3.3 V from U9, only with VBUS (datasheet 6.4)"
- note added: "a 2N7002 that holds the amplifier's EN low while the host sleeps (2 mA -> < 1 uA); the codec itself stays enumerated and draws its suspend current."
- note added: "battery)."
- note added: "coupling capacitors, 0 dB gain (-6 dB with JP3 closed, for very sensitive earphones). Inputs single-ended through 1 uF (8 Hz); EN about 50 ms after"
- note added: "is pulled) and off at once through a Schottky. The switch's output discharge goes through 1k (TPS22919 9.2.2.2): the 5 V falls in about 3 ms, so"
- note added: "the amplifier is off before the codec loses its supply (TPA6132A2 p.12, no pop)."
- note added: "the supply (1M + 100 nF from P1.02, into the pin through 33k: EN may not exceed VDD + 0.3 V, and C137 still holds 3.3 V for a moment when the cable"
- note removed: "1. Second AP2112K (switched 3.3 V for external devices, P0.12 enable) omitted: nothing external to power."
- note removed: "11. C108 1 uF at the regulator output and C109 100 nF at the module: the 10 uF C103 sits at the module's supply pins (VDD / VDDH), 25 mm away. C102 on VIN is 1 uF instead of 10 uF: together they keep the capacitance charged at USB attach near USB 2.0's 10 uF."
- note removed: "3. Microphone: bias 1.2k + 2.2k (demo board 2.2k + 8.2k, for PC microphones) for phone headsets (Android: 1.8-2.9 V through 2.2k); 1k in series before"
- note removed: "4. The demo board's two 10 nF capacitors DVDD - DREG18 and DVDD - DREG33 ('close to IC', for ESD) are fitted."
- note removed: "5 V falls in about 3 ms, so the amplifier is off before the codec loses its supply (TPA6132A2 p.12, no pop)."
- note removed: "5. The amplifier's SGND (pin 15) is grounded at the amplifier (its ground pad and a via into the top ground plane), not on a track of its own to the"
- note removed: "6. The four mode jumpers are also strapped with 10k (MODE/ADSEL low, PWRSEL/MSEL high to DREG33) on top of the chip's internal pulls. D105-D107 are"
- note removed: "C107: VBUS bypass (deviation 10)"
- note removed: "after the supply (1M + 470 nF from P1.02) and off at once through a Schottky. The switch's output discharge goes through 1k (TPS22919 9.2.2.2): the"
- note removed: "coupling capacitors, 0 dB gain (-6 dB with JP3 closed, for very sensitive earphones). Inputs single-ended through 1 uF (8 Hz); EN about 0.25 s"
