File: production/kicad/schematic/lira.kicad_sch (KiCad schematic)
At the start: 211 parts, among them J1 USB-C, J2 battery JST-PH, J3 PJ-320D-4A, Q1 SI2301CDS, SW1 7, SW10 T, SW101 JS102011SAQN, SW102 reset, SW11 Y, SW12 U, SW13 I, SW14 O, SW15 P, SW16 \, SW17 delete, SW18 4, SW19 5, SW2 8, SW20 6, SW21 +, SW22 tab, SW23 A, SW24 S, SW25 D, SW26 F, SW27 G, SW28 H, SW29 J, SW3 9, SW30 K, SW31 L, SW32 ;, SW33 return, SW34 1, SW35 2, SW36 3, SW37 enter, SW38 shift, SW39 Z, SW4 −, SW40 X, SW41 C, SW42 V, SW43 B, SW44 N, SW45 M, SW46 ,, SW47 ., SW48 shift, SW49 fn, SW5 esc, SW50 0, SW51 ., SW52 option, SW53 ⌘, SW54 space, SW55 space, SW56 ⌘, SW57 option, SW6 Q, SW7 W, SW8 E, SW9 R, U1 E73-2G4M08S1C, U2 MCP73831, U3 AP2112K-3.3, U4 USBLC6-2SC6, U5 CH334P, U6 CM108B, U7 TPA6132A2, U8 TPS22919, Y1 32.768kHz, Y2 12MHz

Commit message: rp2040: complete the wired variant (RP2040, USB only, no battery)
Same keyboard, case, plate, sound card and keymap as main; the nRF52840 module, battery, charger,
power path and power switch are replaced by a Raspberry Pi RP2040 with its minimum circuit.

- circuit: RP2040 per "Hardware design with RP2040" (ABM8-272-T3 12 MHz, 2 x 15 pF, 1k on XOUT;
  W25Q128JV, SOIC-8 208 mil; 100 nF per supply pin, 1 uF on VREG_VIN/VOUT; BOOT and RESET
  buttons; 27 ohm USB series); fixes from the WIP: VREG_VIN was unconnected, flash footprint was
  150 mil. Sound card identical to main except the TPS22919 ON / amp EN network driven by VBUS
  (keeps the soft start), refs aligned with main
- PCB: new RP2040 block placement; Fine net class (0.2 mm) for the 0.4 mm-pitch pads, matrix lines
  widened back to 0.3 mm after routing; pre-drawn core supply (under the chip), SWD lines, hub
  crystal, amp VDD and load-switch ground; DRC 0 violations, 0 unconnected
- finish_pcb: removed vias kept alive (SWIG use-after-free), geometric via pruning; gen_pcb: no
  stale .kicad_pro loaded, so a rebuild equals a clean build
- schematic regenerated (ERC 0 errors), netlist match; independent checker extended for the
  RP2040 (Q01-Q12): 42 PASS, 0 FAIL, 3 WARN; main's netlist unchanged
- case: no battery pocket, paperclip hole to BOOT; fit check 0 FAIL, 3 WARN (as main)
- firmware: RMK 0.9 + Vial on the RP2040 (embassy-rp, boot2 W25Q080), no BLE / audio gate
- docs: README, build guide, source README, production regenerated; usb/ scaffold folded in
Parts:
- removed C101: 10uF, Capacitor_SMD:C_0603_1608Metric, symbol Device:C
- removed C104: 10nF, Capacitor_SMD:C_0603_1608Metric, symbol Device:C
- removed C105, C106: 18pF, Capacitor_SMD:C_0603_1608Metric, symbol Device:C
- removed C107: 4.7uF, Capacitor_SMD:C_0603_1608Metric, symbol Device:C
- removed C109: 100nF, Capacitor_SMD:C_0603_1608Metric, symbol Device:C
- removed D101: B5819W, Diode_SMD:D_SOD-123, symbol Device:D_Schottky
- removed D102: LED white, LED_SMD:LED_0603_1608Metric, symbol Device:LED
- removed J2: battery JST-PH, Connector_JST:JST_PH_S2B-PH-SM4-TB_1x02-1MP_P2.00mm_Horizontal, symbol Connector:Conn_01x02_Pin
- removed JP1: charge 200 mA, Jumper:SolderJumper-2_P1.3mm_Open_RoundedPad1.0x1.5mm, symbol Jumper:SolderJumper_2_Open
- removed JP2: switch bypass, Jumper:SolderJumper-2_P1.3mm_Open_RoundedPad1.0x1.5mm, symbol Jumper:SolderJumper_2_Open
- removed Q1: SI2301CDS, Package_TO_SOT_SMD:SOT-23, symbol Transistor_FET:AO3401A
- removed R101, R117: 100k, Resistor_SMD:R_0603_1608Metric, symbol Device:R
- removed R102: 1k, Resistor_SMD:R_0603_1608Metric, symbol Device:R
- removed R103, R104: 10k, Resistor_SMD:R_0603_1608Metric, symbol Device:R
- removed R105, R106: 10M, Resistor_SMD:R_0603_1608Metric, symbol Device:R
- removed SW101: JS102011SAQN, Button_Switch_SMD:SW_SPDT_CK_JS102011SAQN, symbol Switch:SW_SPDT
- removed TP7: VBAT, TestPoint:TestPoint_Pad_D1.5mm, symbol Connector:TestPoint
- removed TP8: VIN, TestPoint:TestPoint_Pad_D1.5mm, symbol Connector:TestPoint
- removed U1: E73-2G4M08S1C, lcsc:WIRELM-SMD_E73-2G4M08S1C, symbol lira:E73
- removed U2: MCP73831, Package_TO_SOT_SMD:SOT-23-5, symbol lira:MCP73831
- removed Y1: 32.768kHz, Crystal:Crystal_SMD_3215-2Pin_3.2x1.5mm, symbol Device:Crystal
- added C1, C10, C15, C2, C3, C4, C5, C6, C7, C8, C9: 100nF, Capacitor_SMD:C_0603_1608Metric, symbol Device:C
- added C11, C12: 1uF, Capacitor_SMD:C_0603_1608Metric, symbol Device:C
- added C13, C14: 15pF, Capacitor_SMD:C_0603_1608Metric, symbol Device:C
- added R1, R3: 1k, Resistor_SMD:R_0603_1608Metric, symbol Device:R
- added R2, R4: 10k, Resistor_SMD:R_0603_1608Metric, symbol Device:R
- added R5, R6: 27, Resistor_SMD:R_0603_1608Metric, symbol Device:R
- added SW101: BOOT, lcsc:SW-SMD_4P-L5.1-W5.1-P3.70-LS6.5-TL_H1.5, symbol lira:SW_PUSH_4
- added U1: RP2040, Package_DFN_QFN:QFN-56-1EP_7x7mm_P0.4mm_EP3.2x3.2mm, symbol lira:RP2040
- added U2: W25Q128JVS, Package_SO:SOIC-8_5.3x5.3mm_P1.27mm, symbol Memory_Flash:W25Q128JVS
- added Y1: 12MHz, Crystal:Crystal_SMD_3225-4Pin_3.2x2.5mm, symbol Device:Crystal_GND24
- SW102: value reset -> RESET
Connections:
- net AUD_EN is gone; now on net VBUS: D104.1 (K), R113.1, U8.3 (ON)
- net VIN is gone; now on net VBUS: C102.1, U3.1 (VIN), U3.3 (EN)
- net 3V3: now also C1.1, C11.1, C15.1, C2.1, C3.1, C4.1, C5.1, C6.1, C7.1, C8.1, R2.1, R4.1, U1.1 (IOVDD), U1.10 (IOVDD), U1.22 (IOVDD), U1.33 (IOVDD), U1.42 (IOVDD), U1.43 (ADC_AVDD), U1.44 (VREG_VIN), U1.48 (USB_VDD), U1.49 (IOVDD), U2.8 (VCC)
- net COL0: now also U1.38 (GPIO26/ADC0)
- net COL1: now also U1.37 (GPIO25)
- net COL10: now also U1.8 (GPIO6)
- net COL11: now also U1.6 (GPIO4)
- net COL12: now also U1.5 (GPIO3)
- net COL13: now also U1.4 (GPIO2)
- net COL14: now also U1.3 (GPIO1)
- net COL15: now also U1.2 (GPIO0)
- net COL16: now also U1.7 (GPIO5)
- net COL2: now also U1.36 (GPIO24)
- net COL3: now also U1.35 (GPIO23)
- net COL4: now also U1.34 (GPIO22)
- net COL5: now also U1.32 (GPIO21)
- net COL6: now also U1.14 (GPIO11)
- net COL7: now also U1.12 (GPIO9)
- net COL8: now also U1.11 (GPIO8)
- net COL9: now also U1.9 (GPIO7)
- net GND: now also C1.2, C10.2, C11.2, C12.2, C13.2, C14.2, C15.2, C2.2, C3.2, C4.2, C5.2, C6.2, C7.2, C8.2, C9.2, SW101.4, U1.19 (TESTEN), U1.57 (GND), U2.4 (GND), Y1.2 (G), Y1.4 (G)
- net LED_RED: now also U1.39 (GPIO27/ADC1)
- net MCU_DN: now also R6.2
- net MCU_DP: now also R5.2
- net RESET: now also R4.2, U1.26 (RUN)
- net ROW0: now also U1.13 (GPIO10)
- net ROW1: now also U1.31 (GPIO20)
- net ROW2: now also U1.29 (GPIO18)
- net ROW3: now also U1.30 (GPIO19)
- net SWCLK: now also U1.24 (SWCLK)
- net SWDIO: now also U1.25 (SWDIO)
- new net 1V1: C10.1, C12.1, C9.1, U1.23 (DVDD), U1.45 (VREG_VOUT), U1.50 (DVDD)
- new net BOOT: R3.2, SW101.1
- new net QSPI_SCLK: U1.52 (QSPI_SCLK), U2.6 (CLK)
- new net QSPI_SD0: U1.53 (QSPI_SD0), U2.5 (DI/IO_{0})
- new net QSPI_SD1: U1.55 (QSPI_SD1), U2.2 (DO/IO_{1})
- new net QSPI_SD2: U1.54 (QSPI_SD2), U2.3 (~{WP}/IO_{2})
- new net QSPI_SD3: U1.51 (QSPI_SD3), U2.7 (~{HOLD}/~{RESET}/IO_{3})
- new net QSPI_SS: R2.2, R3.1, U1.56 (QSPI_SS), U2.1 (~{CS})
- new net RP_DN: R6.1, U1.46 (USB_DM)
- new net RP_DP: R5.1, U1.47 (USB_DP)
- new net XIN: C13.1, U1.20 (XIN), Y1.1
- new net XOUT: R1.1, U1.21 (XOUT)
- new net XOUT_X: C14.1, R1.2, Y1.3
- no-connect marks 44 -> 47
Other:
- note added: "1. Supply: VBUS through a TPS22919 load switch (soft start 1.3 ms, output discharge) to AUD_5V, ON tied to VBUS (the wireless board drives it from a"
- note added: "1. USB only, no battery: no Ebyte E73 (nRF52840) module, no Bluetooth, no Li-Po cell, no charger (MCP73831), no power path (B5819W + SI2301), no power switch, no battery divider, no 32.768 kHz crystal, no antenna keep-out."
- note added: "12 MHz crystal ABM8-272-T3 (CL 10 pF): 2 x 15 pF, 1k on XOUT; QSPI flash W25Q128JV, /CS pulled up"
- note added: "2. Raspberry Pi RP2040 instead of the module, with the minimum circuit of Raspberry Pi's 'Hardware design with RP2040' (the Pico's): 12 MHz crystal ABM8-272-T3 (the one Raspberry Pi qualified) with 2 x 15 pF and 1k in series on XOUT; W25Q128JV QSPI flash (16 MB) with a 10k pull-up on QSPI_SS; 100 nF on each of the six IOVDD pins, on both DVDD, USB_VDD and ADC_AVDD, 1 uF on"
- note added: "3. USB: hub port 3 goes to the RP2040's USB_DP / USB_DM through 27 ohm series resistors (as on the Pico and in the design guide), instead of the module's D+ / D-."
- note added: "3.3 V regulator AP2112K from VBUS (EN tied to VIN); 10 uF bulk at the RP2040"
- note added: "4. Programming: the RP2040's boot ROM is a USB drive (RPI-RP2) - no bootloader to flash with an SWD probe. A blank board starts in it; BOOT (SW101, QSPI_SS to GND through 1k) held while plugging the cable enters it again; RESET (SW102) pulls RUN low. The SWD pads stay for debugging."
- note added: "5. 3.3 V regulator AP2112K-3.3 (the same as the wireless board) fed straight from VBUS: 1 uF in, 1 uF + 10 uF out."
- note added: "6. Status LED (red, Caps Lock) on an RP2040 GPIO, through 1k, as on the wireless board."
- note added: "7. Test points: SWD (SWCLK, SWDIO, RESET, GND) in one row in front of the RP2040, 3V3 behind it, VBUS; no VBAT / VIN."
- note added: "8. Sound card: the supply switch U8 is turned on by VBUS instead of a GPIO (the wireless board has it on only in USB mode; here it always is) and its pull-down is dropped. It still soft-starts the sound card's 5 V: its 17 uF are charged through the switch's controlled rise, not straight from the cable (only ~3 uF sit directly on VBUS). The amplifier's EN delay (1M + 470 nF)"
- note added: "BOOT: QSPI_SS to GND through 1k (USB boot ROM); RESET: RUN to GND, 10k pull-up"
- note added: "GPIO, on only in USB mode): the sound card's capacitors are charged slowly after the cable has made contact. A hard switch-on would dip VBUS enough"
- note added: "Lira, wired: Raspberry Pi RP2040, USB-C only (no battery), 57 keys, built-in USB sound card"
- note added: "RP2040 decoupling: 100 nF at each IOVDD, USB_VDD, ADC_AVDD and DVDD pin; 1 uF at VREG_VIN and VREG_VOUT"
- note added: "Raspberry Pi RP2040 (1.1 V core from its own regulator: VREG_VOUT -> DVDD); USB through 27 ohm to the hub's port 3; status LED (Caps Lock) on a GPIO; SWD pads"
- note added: "Sound card supply: TPS22919 load switch, turned on by VBUS (soft start); headphone amplifier TPA6132A2 (DirectPath, 0 dB; -6 dB with JP3 closed); headset jack, CTIA"
- note added: "Supplies: VBUS from the receptacle, codec supplies from VBUS through ferrite beads"
- note added: "The wireless board (branch main: nRF52840 module, Li-Po) with the radio and the battery taken out; the RP2040 follows Raspberry Pi's 'Hardware design with RP2040' (the Pico's circuit). Differences from the wireless board:"
- note added: "VREG_VIN and VREG_VOUT; the internal regulator makes the 1.1 V core supply; TESTEN grounded."
- note added: "after the supply (1M + 470 nF from VBUS), and dragged down with VBUS through a Schottky when the cable is pulled (EN stays within a Schottky drop"
- note added: "coupling capacitors, 0 dB gain (-6 dB with JP3 closed, for very sensitive earphones). Inputs single-ended through 1 uF (8 Hz); EN about 0.15 s"
- note added: "of VBUS). On unplug the codec and the amplifier lose their supply together: listen for a click."
- note added: "runs from VBUS too, and D104 drags EN down with VBUS on unplug."
- note added: "to reset the hub (CH334 datasheet 6.1)."
- note added: "upstream from the receptacle, port 3 -> RP2040, port 2 -> codec"
- note removed: "1. Second AP2112K (switched 3.3 V for external devices, P0.12 enable) omitted: nothing external to power."
- note removed: "1. Supply: VBUS through a TPS22919 load switch (soft start 1.3 ms, output discharge) to AUD_5V, ON = P1.02 with a 100k pull-down: the sound card is"
- note removed: "10. C107 4.7 uF added on VBUS at the charger's VDD pin (the MCP73831 datasheet asks for 4.7 uF; Nordic's reference circuit has 4.7 uF on VBUS; the BlueMicro840 has none)."
- note removed: "11. C108 1 uF at the regulator output and C109 100 nF at the module: the 10 uF C103 sits at the module's supply pins (VDD / VDDH), 25 mm away. C102 on VIN is 1 uF instead of 10 uF: together they keep the capacitance charged at USB attach near USB 2.0's 10 uF."
- note removed: "12. Charger MCP73831 instead of the TP4054, same pins and same PROG resistor (1000 V / R_PROG): it is stable with no battery, so the board also works when built without one (its STAT pin, and the white LED, stay off)."
- note removed: "13. Battery divider 10M + 10M with 10 nF (BlueMicro840: 806k + 2M, 1 nF): the MCP73831 recognises a missing battery only if VBAT sees more than 7 MOhm (datasheet 4.2); 10 nF >= 2^12 x the SAADC's 2.5 pF keeps the reading within 1 LSB (Nordic, 'Measuring Lithium battery voltage with nRF52'), and RMK samples it every 30 s. Drain 0.2 uA."
- note removed: "14. Built-in USB sound card: the USB-C data lines go (through the ESD array) to a CH334P hub; hub port 3 goes to the module's D+ / D-, port 2 to a CM108B codec (C-Media demo board v1.33) with a 3.5 mm headset jack."
- note removed: "2. USBLC6-2SC6 ESD array added on D+ / D- / VBUS at the USB-C receptacle."
- note removed: "3. Power switch SW101 (C&K JS102011SAQN, 300 mA) in the battery + line, as on ZMK keyboards; JP2 bypasses it."
- note removed: "3.3 V regulator (BlueMicro840 U3, EN tied to VIN) and 32.768 kHz crystal (BlueMicro840 Y2 C1 C2)"
- note removed: "4. JP1 + R104: closing the solder jumper puts a second 10k on PROG: charge current 100 mA -> 200 mA."
- note removed: "5 V falls in about 3 ms, so the amplifier is off before the codec loses its supply (TPA6132A2 p.12, no pop)."
- note removed: "5. Reset push button SW102 to GND (the BlueMicro840 has only a test point)."
- note removed: "6. USB-C shield pads to GND (left open on the BlueMicro840)."
- note removed: "7. LEDs: charging LED white, status LED red on P1.04 only (BlueMicro840: green charging, red P1.04, blue P1.10)."
- note removed: "8. DCCH inductor pads (DNP on the BlueMicro840) not fitted at all; P1.10 is a free GPIO here, P1.02 switches the sound card."
- note removed: "9. Test points added on VBUS, VBAT and VIN (BlueMicro840: SWDIO, SWCLK, VCC, GND, RESET, P1.02)."
- note removed: "Battery: JST-PH, power switch (JP2 bypasses it), divider 10M / 10M + 10nF into P0.31 (BlueMicro840 R4 R6 C6: 806k / 2M + 1nF)"
- note removed: "C103, C109: at the module's VDD / VDDH pins"
- note removed: "C107: VBUS bypass (deviation 10)"
- note removed: "Charger MCP73831 (BlueMicro840 U4 is a TP4054, same pins): 100 mA, 200 mA with JP1 closed; white LED on while charging"
- note removed: "Lira: nRF52840 (Ebyte E73-2G4M08S1C), USB-C + Li-Po, 57 keys, built-in USB sound card"
- note removed: "Power / USB / programming copied from the BlueMicro840 (jpconstantineau/NRF52-Board), a board built with this module, assembled by JLCPCB and sold. Differences from it:"
- note removed: "Power path: USB through the Schottky, battery through the P-MOSFET (off while VBUS is present)"
- note removed: "R101: VBUS bleeder (BlueMicro840 R3)"
- note removed: "Sound card supply: TPS22919 load switch, on only in USB mode (P1.02); headphone amplifier TPA6132A2 (DirectPath, 0 dB; -6 dB with JP3 closed); headset jack, CTIA"
- note removed: "Supplies: VBUS from the receptacle, BAT+ from the cell, VIN from the power path, codec supplies from VBUS through ferrite beads"
- note removed: "after the supply (1M + 470 nF from P1.02) and off at once through a Schottky. The switch's output discharge goes through 1k (TPS22919 9.2.2.2): the"
- note removed: "coupling capacitors, 0 dB gain (-6 dB with JP3 closed, for very sensitive earphones). Inputs single-ended through 1 uF (8 Hz); EN about 0.25 s"
- note removed: "nRF52840 module, normal-voltage mode (VDD = VDDH = 3.3 V); reset button; status LED on P1.04 (bootloader LED); SWD pads"
- note removed: "powered only in USB mode (firmware src/audio_gate.rs). A hard switch-on would dip VBUS enough to reset the hub (CH334 datasheet 6.1)."
- note removed: "upstream from the receptacle, port 3 -> module, port 2 -> codec"
- title: Lira -> Lira (wired)

Commit message: Fix placement data, silkscreen, firmware and docs
Supply and placement (blocking before an order):
- Hot-swap socket C2803348 is discontinued (0 stock): replaced by C41430893
  in the BOM, schematic, netlist and checks
- cpl.csv: rotations converted to JLCPCB's convention (per-part LCSC
  footprint angle, bottom side 180 - angle) and origin offsets for J1 and J3

Board (silkscreen only; tracks, vias and placement unchanged, DRC 0 errors):
- every label >= 1.0 mm; SWD pad names beside the pads, CAPS beside its LED,
  -6dB below its jumper, board name

Firmware:
- RMK 0.9.0 patched at build time (firmware/patch_rmk.py, SHA-256 checked):
  the matrix waits for the rows to fall before the next column (weak RP2040
  pull-downs, long rows: a held key could show up in the next column), and
  USB asks for 100 mA instead of 450 mA
- random Vial keyboard UID; Cargo.toml metadata

Build: one datasheet check made deterministic.

Docs: README, guide and production README corrected (screws, ears, print
orientation, JLCPCB Economic assembly, stock warning, bench checks,
licences) and
Parts:
- SW1, SW10, SW11, SW12, SW13, SW14, SW15, SW16, SW17, SW18, SW19, SW2, SW20, SW21, SW22, SW23, SW24, SW25, SW26, SW27, SW28, SW29, SW3, SW30, SW31, SW32, SW33, SW34, SW35, SW36, SW37, SW38, SW39, SW4, SW40, SW41, SW42, SW43, SW44, SW45, SW46, SW47, SW48, SW49, SW5, SW50, SW51, SW52, SW53, SW54, SW55, SW56, SW57, SW6, SW7, SW8, SW9: LCSC C2803348 -> C41430893

Commit message: Rework the board placement and routing
- RP2040: 0402 decoupling at the pins, every supply connection drawn on the
  bottom layer (corner bus for VREG_VIN / ADC_AVDD / IOVDD 42, IOVDD 1-10-22 and
  33-42 tied inside the pin ring, 1.1 V ring under the package), top layer kept
  free of tracks over the package, its capacitors and its crystal; crystal at the
  front pins; 27 ohm USB resistors at the chip; QSPI lines and 3.3 V links drawn
- Exposed pad: four tented vias at the corners, paste in five windows clear of them
- Hub on 3.3 V (V5 = VDD33); SMF5.0A TVS and 4.7 uF damped by 1 ohm at the
  receptacle; VBUS divider on GPIO29 (ADC3)
- Sound card switch on GPIO12, amplifier EN on GPIO13; firmware (sound_card.rs)
  turns the card on when configured, the amplifier off in suspend and on VBUS
  fall; async_matrix; RMK patch v2 settles the rows after the async wake
- 100 nF at each CM108B AVDD pin; jack ESD clamps between the jack and the ferrites
- New checks: V01 (VBUS protection), V02 (VBUS sense), G01 (layout distances,
  pcb/layout_metrics.py); Q12 budgets the hub at 85 mA
- DRC 0 / 0 unconnected, ERC 0 errors, netlist match, 45 PASS 0 FAIL 3 WARN,
  fit check 0 FAIL; production files, renders and docs regenerated
Parts:
- removed C10, C2, C4, C7: 100nF, Capacitor_SMD:C_0603_1608Metric, symbol Device:C
- removed C111: 10uF, Capacitor_SMD:C_0603_1608Metric, symbol Device:C
- removed C137: 470nF, Capacitor_SMD:C_0603_1608Metric, symbol Device:C
- removed D104: B5819W, Diode_SMD:D_SOD-123, symbol Device:D_Schottky
- added C104: 4.7uF, Capacitor_SMD:C_0805_2012Metric, symbol Device:C
- added C140: 100nF, Capacitor_SMD:C_0402_1005Metric, symbol Device:C
- added C16: 1nF, Capacitor_SMD:C_0603_1608Metric, symbol Device:C
- added D108: SMF5.0A, Diode_SMD:D_SOD-123F, symbol Device:D_Zener
- added R119, R124: 100k, Resistor_SMD:R_0603_1608Metric, symbol Device:R
- added R7: 1, Resistor_SMD:R_0603_1608Metric, symbol Device:R
- added R8: 22k, Resistor_SMD:R_0603_1608Metric, symbol Device:R
- added R9: 27k, Resistor_SMD:R_0603_1608Metric, symbol Device:R
- C1, C3, C5, C6, C8, C9: footprint Capacitor_SMD:C_0603_1608Metric -> Capacitor_SMD:C_0402_1005Metric; LCSC C14663 -> C1525
- C103: value 10uF -> 4.7uF; LCSC C19702 -> C19666
- C11, C12: footprint Capacitor_SMD:C_0603_1608Metric -> Capacitor_SMD:C_0402_1005Metric; LCSC C15849 -> C52923
- C13, C14: footprint Capacitor_SMD:C_0603_1608Metric -> Capacitor_SMD:C_0402_1005Metric; LCSC C1644 -> C1548
- R1: footprint Resistor_SMD:R_0603_1608Metric -> Resistor_SMD:R_0402_1005Metric; LCSC C21190 -> C11702
- R5, R6: footprint Resistor_SMD:R_0603_1608Metric -> Resistor_SMD:R_0402_1005Metric; LCSC C25190 -> C2909343
Connections:
- net HUB_3V3 is gone; now on net 3V3: C112.1, U5.16 (VDD33)
- net 3V3: now also C110.1, U5.15 (V5)
- net AMP_EN: now also R113.1, R124.2; no longer R113.2
- net AUD_AVDD: now also C140.1
- net GND: now also R113.2, C104.2, C140.2, C16.2, D108.2 (A), R119.2, R9.2
- net VBUS: now also D108.1 (K), R7.1, R8.1; no longer C110.1, R113.1, U5.15 (V5), U8.3 (ON)
- net AUD_EN: now reaches U1.15 (GPIO12)
- net AUD_EN: now also U8.3 (ON), R119.1
- net AMP_ON: now reaches U1.16 (GPIO13)
- net AMP_ON: now also R124.1
- net VBUS_SENSE: now reaches U1.41 (GPIO29/ADC3)
- net VBUS_SENSE: now also C16.1, R8.2, R9.1
- new net VBUS_DAMP: C104.1, R7.2
- no-connect marks 47 -> 44
Other:
- note added: "1. Supply: VBUS through a TPS22919 load switch (soft start 1.3 ms, output discharge) to AUD_5V, ON from an RP2040 GPIO (on once the host has"
- note added: "2. Raspberry Pi RP2040 instead of the module, with the minimum circuit of Raspberry Pi's 'Hardware design with RP2040' (the Pico's): 12 MHz crystal ABM8-272-T3 (the one Raspberry Pi qualified) with 2 x 15 pF and 1k in series on XOUT; W25Q128JV QSPI flash (16 MB) with a 10k pull-up on QSPI_SS; 100 nF (0402) on IOVDD 1, 22, 42, 49, on DVDD 23 and on ADC_AVDD, USB_VDD sharing"
- note added: "3.3 V regulator AP2112K from VBUS (EN tied to VIN), also for the hub; 4.7 uF bulk at the RP2040"
- note added: "4. The demo board's two 10 nF capacitors DVDD - DREG18 and DVDD - DREG33 ('close to IC', for ESD) are fitted; each AVDD pin (29, 34) has its own 100"
- note added: "5. 3.3 V regulator AP2112K-3.3 (the same as the wireless board) fed straight from VBUS: 1 uF in, 1 uF + 4.7 uF out; it also supplies the USB hub (V5 and VDD33 on 3.3 V, CH334 datasheet 6.4), so nothing but the regulator, the sound card's switch and the protection sits on VBUS."
- note added: "6. VBUS protection at the receptacle: SMF5.0A TVS and a 4.7 uF bulk capacitor damped by 1 ohm (hot-plug ringing); VBUS divider 22k / 27k + 1 nF to GPIO29 (ADC3) for the firmware."
- note added: "6.1)."
- note added: "7. Status LED (red, Caps Lock) on an RP2040 GPIO, through 1k, as on the wireless board."
- note added: "8. Test points: SWD (SWCLK, SWDIO, RESET, GND) in one row in front of the RP2040, 3V3 behind it, VBUS; no VBAT / VIN."
- note added: "9. Sound card: the supply switch U8 is on a GPIO (GPIO12) with a 100k pull-down, as on the wireless board; the headphone amplifier's EN has its own GPIO (GPIO13) through 100k, held low by 1M (the wireless board delays it with an RC from the switch). The firmware turns the sound card on when the host has configured the keyboard, the amplifier 0.2 s later, the amplifier off in"
- note added: "GPIO through 100k (1M to ground): on 0.2 s after the supply, off in USB suspend (2 mA saved) and, when the cable is pulled, as soon as the firmware"
- note added: "IOVDD 49's as in the design guide, IOVDD 10 / 33 sharing 1's / 42's through a tie under the package and DVDD 50 VREG_VOUT's 1 uF through the 1.1 V ring under it; 1 uF on VREG_VIN and VREG_VOUT; each within a few mm of its pin on the bottom layer; the internal regulator makes the 1.1 V core supply; TESTEN grounded."
- note added: "RESET#, PGANG and ports 1 / 4 left open; V5 and VDD33 on the 3.3 V rail (datasheet 6.4)"
- note added: "RP2040 decoupling: 100 nF at IOVDD 1, 22, 42, 49, ADC_AVDD and DVDD 23 (USB_VDD shares 49's, IOVDD 10 / 33 1's / 42's, DVDD 50 VREG_VOUT's 1 uF); 1 uF at VREG_VIN and VREG_VOUT"
- note added: "Sound card supply: TPS22919 load switch, on from GPIO12 (soft start); headphone amplifier TPA6132A2 (DirectPath, 0 dB; -6 dB with JP3 closed), EN from GPIO13; headset jack, CTIA"
- note added: "USB suspend and as soon as VBUS starts to fall."
- note added: "USB-C (sink: 5.1k on each CC), ESD protection, VBUS TVS and damped bulk capacitor"
- note added: "VBUS sense: 22k / 27k + 1 nF to GPIO29 (ADC3)"
- note added: "bidirectional ESD clamps (PESD5V0S1BA) on the jack's left, right and microphone contacts, between the jack and the ferrites, each with its own"
- note added: "configured the keyboard): the sound card's capacitors are charged slowly. A hard switch-on would dip VBUS enough to reset the hub (CH334 datasheet"
- note added: "coupling capacitors, 0 dB gain (-6 dB with JP3 closed, for very sensitive earphones). Inputs single-ended through 1 uF (8 Hz); EN from an RP2040"
- note added: "ground via: a DirectPath output swings below GND, so the clamp must be bidirectional."
- note added: "nF."
- note added: "sees VBUS fall, before the codec loses its supply (no click)."
- note removed: "1. Supply: VBUS through a TPS22919 load switch (soft start 1.3 ms, output discharge) to AUD_5V, ON tied to VBUS (the wireless board drives it from a"
- note removed: "2. Raspberry Pi RP2040 instead of the module, with the minimum circuit of Raspberry Pi's 'Hardware design with RP2040' (the Pico's): 12 MHz crystal ABM8-272-T3 (the one Raspberry Pi qualified) with 2 x 15 pF and 1k in series on XOUT; W25Q128JV QSPI flash (16 MB) with a 10k pull-up on QSPI_SS; 100 nF on each of the six IOVDD pins, on both DVDD, USB_VDD and ADC_AVDD, 1 uF on"
- note removed: "3.3 V regulator AP2112K from VBUS (EN tied to VIN); 10 uF bulk at the RP2040"
- note removed: "4. The demo board's two 10 nF capacitors DVDD - DREG18 and DVDD - DREG33 ('close to IC', for ESD) are fitted."
- note removed: "5. 3.3 V regulator AP2112K-3.3 (the same as the wireless board) fed straight from VBUS: 1 uF in, 1 uF + 10 uF out."
- note removed: "6. Status LED (red, Caps Lock) on an RP2040 GPIO, through 1k, as on the wireless board."
- note removed: "7. Test points: SWD (SWCLK, SWDIO, RESET, GND) in one row in front of the RP2040, 3V3 behind it, VBUS; no VBAT / VIN."
- note removed: "8. Sound card: the supply switch U8 is turned on by VBUS instead of a GPIO (the wireless board has it on only in USB mode; here it always is) and its pull-down is dropped. It still soft-starts the sound card's 5 V: its 17 uF are charged through the switch's controlled rise, not straight from the cable (only ~3 uF sit directly on VBUS). The amplifier's EN delay (1M + 470 nF)"
- note removed: "GPIO, on only in USB mode): the sound card's capacitors are charged slowly after the cable has made contact. A hard switch-on would dip VBUS enough"
- note removed: "RESET#, PGANG and ports 1 / 4 left open"
- note removed: "RP2040 decoupling: 100 nF at each IOVDD, USB_VDD, ADC_AVDD and DVDD pin; 1 uF at VREG_VIN and VREG_VOUT"
- note removed: "Sound card supply: TPS22919 load switch, turned on by VBUS (soft start); headphone amplifier TPA6132A2 (DirectPath, 0 dB; -6 dB with JP3 closed); headset jack, CTIA"
- note removed: "USB-C (sink: 5.1k on each CC) and ESD protection"
- note removed: "VREG_VIN and VREG_VOUT; the internal regulator makes the 1.1 V core supply; TESTEN grounded."
- note removed: "after the supply (1M + 470 nF from VBUS), and dragged down with VBUS through a Schottky when the cable is pulled (EN stays within a Schottky drop"
- note removed: "be bidirectional."
- note removed: "bidirectional ESD clamps (PESD5V0S1BA) on the jack's left, right and microphone contacts: a DirectPath output swings below GND, so the clamp must"
- note removed: "coupling capacitors, 0 dB gain (-6 dB with JP3 closed, for very sensitive earphones). Inputs single-ended through 1 uF (8 Hz); EN about 0.15 s"
- note removed: "of VBUS). On unplug the codec and the amplifier lose their supply together: listen for a click."
- note removed: "runs from VBUS too, and D104 drags EN down with VBUS on unplug."
- note removed: "to reset the hub (CH334 datasheet 6.1)."
